File: kicad_frame_strip_v1/framePCB.sch (KiCad schematic (older format))
At the start: 60 parts, among them J1 dc_jack, J2 BOOT, J3 VIN/GRB0, J4 VIN/GRB1, J5 VIN/RGB2, J6 USART, J7 JST, J8 VDD, Q1 MOS_N_GDS, Q2 MOS_N_GDS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

Commit message: Version 3 PCB
Parts:
- D1, D2, D3, D4, D5, D6: symbol LED -> LED-RESCUE-framePCB
- RV1, RV2, RV3: symbol POT -> POT-RESCUE-framePCB
Changed lines of the file:
@@
 EESchema Schematic File Version 2
+LIBS:framePCB-rescue
 LIBS:power
 LIBS:device
@@
 LIBS:memory
 LIBS:xilinx
-LIBS:special
 LIBS:microcontrollers
 LIBS:dsp
@@
 LIBS:valves
 LIBS:crf_1
-LIBS:w_freaquency
+LIBS:freakuency
+LIBS:w_analog
 LIBS:w_connectors
 LIBS:w_device
+LIBS:w_logic
+LIBS:w_memory
+LIBS:w_microcontrollers
+LIBS:w_opto
+LIBS:Worldsemi
+LIBS:w_relay
+LIBS:w_rtx
 LIBS:w_transistor
+LIBS:w_vacuum
 LIBS:framePCB-cache
 EELAYER 25 0
@@
 $EndComp
 $Comp
-L POT RV1
+L POT-RESCUE-framePCB RV1
 U 1 1 56327631
 P 5400 7900
@@
 $EndComp
 $Comp
-L POT RV2
+L POT-RESCUE-framePCB RV2
 U 1 1 563299A7
 P 5700 7900
@@
 GND
 $Comp
-L LED D1
+L LED-RESCUE-framePCB D1
 U 1 1 5632FEA2
 P 1150 7750
@@
 $EndComp
 $Comp
-L LED D2
+L LED-RESCUE-framePCB D2
 U 1 1 563308D1
 P 1450 7750
@@
 $EndComp
 $Comp
-L LED D3
+L LED-RESCUE-framePCB D3
 U 1 1 5633093F
 P 1750 7750
@@
 POT2
 $Comp
-L LED D4
+L LED-RESCUE-framePCB D4
 U 1 1 563324AB
 P 2550 7750
@@
 $EndComp
 $Comp
-L LED D5
+L LED-RESCUE-framePCB D5
 U 1 1 563324C4
 P 2850 7750
@@
 $EndComp
 $Comp
-L LED D6
+L LED-RESCUE-framePCB D6
 U 1 1 563324CA
 P 3150 7750
@@
 Connection ~ 1600 9250
 $Comp
-L GND #PWR03
+L GND-RESCUE-framePCB #PWR03
 U 1 1 5633A332
 P 2350 9250
@@
 En lampa med alla lampor i den
 $Comp
-L POT RV3
+L POT-RESCUE-framePCB RV3
 U 1 1 563689A7
 P 6250 7900
