File: kicad_frame_strip_v2/frame_strip.sch (KiCad schematic (older format))
At the start: 61 parts, among them J1 PROGRAM, J10 HEADER_1, J11 HEADER_1, J12 HEADER_1, J2 USART2, J3 HEADER_4, J4 HEADER_4, J5 HEADER_4, J6 HEADER_2, J7 DC_POWER_JACK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

Commit message: PCB, code
Parts:
- added J13, J14, J15: HEADER_3, w_pin_strip:pin_socket_3, symbol HEADER_3
- added J16: I2C2, w_pin_strip:pin_socket_3, symbol HEADER_3
- added SW4: RESET, w_switch:smd_push, symbol SW_PUSH
- C6: footprint w_smd_cap:c_0603 -> w_smd_cap:c_elec_5x5.3
- LD1: value LED -> LED1
- LD2: value LED -> LED2
- LD3: value LED -> LED3
- LD4: value LED -> LED4
- SW3: value SW_SPDT -> ON/OFF
- renumbered R22 to ADC4, R23 to ADC5, R24 to ADC6
Connections:
- net 12V: now also J7.1, SW3.1 (COM); no longer C6.1, SW3.2 (NC), U6.3 (VIN)
- net GND: now also SW4.1
- net LED1: now also U1.34 (PA13-JTMS-SWDIO/Remap:PA13); no longer U1.41 (PB5-I2C1_SMBA_/_TIM16_BKIN/Remap:TIM3_CH2/SPI1_MOSI)
- net LED2: now also U1.37 (PA14-JTCK/SWCLK/Remap:PA14); no longer U1.21 (PB10-I2C2_SCL/USART3_TX/Remap:TIM2_CH3/HDMI_CEC)
- net LED3: now also U1.38 (PA15-JTDI-Remap:TIM2_CH1_ETR/SPI1_NSS); no longer U1.22 (PB11-I2C2_SDA/USART3_RX/Remap:TIM2_CH4)
- net LED4: now also U1.39 (PB3-JTDO-Remap:TIM2_CH2/PB3/TRACESWO/SPI1_SCK); no longer U1.25 (PB12-SPI2_NSS/I2C2_SMBA/TIM1_BKIN/USART3_CK)
- net RESET: now also SW4.2
- net SPI1_MOSI: now also J8.1; no longer J8.3
- net SPI1_SCK: now also J8.3; no longer J8.1
- net TIM1_CH1: now also J15.3
- net TIM2_CH2: now also J14.2
- net TIM3_CH2: now also J14.3
- net TIM3_CH3: now also J15.1
- net TIM3_CH4: now also J15.2
- net TIM4_CH1: now also J13.1
- net TIM4_CH2: now also J13.2
- net TIM4_CH3: now also J13.3
- net TIM4_CH4: now also J14.1
- new net: C6.1, SW3.2 (NC), U6.3 (VIN)
- new net PB12: J16.3, U1.25 (PB12-SPI2_NSS/I2C2_SMBA/TIM1_BKIN/USART3_CK)
- new net SCL: J16.1, U1.21 (PB10-I2C2_SCL/USART3_TX/Remap:TIM2_CH3/HDMI_CEC)
- new net SDA: J16.2, U1.22 (PB11-I2C2_SDA/USART3_RX/Remap:TIM2_CH4)
- no-connect marks 11 -> 9
Changed lines of the file:
@@
 EESchema Schematic File Version 2
+LIBS:frame_strip-rescue
 LIBS:power
 LIBS:w_analog
@@
 $EndComp
 Wire Wire Line
-	1650 3800 1300 3800
+	1300 3800 2250 3800
 Text Label 1650 3250 0    60   ~ 0
 3.3V
@@
 Text Label 3750 1700 2    60   ~ 0
 ADC1_5
-NoConn ~ 3750 2600
-NoConn ~ 3750 2700
-NoConn ~ 3750 2800
-NoConn ~ 3750 3300
 NoConn ~ 3750 3400
 $Comp
@@
 P 2000 8000
 F 0 "SW3" H 2000 7900 50  0000 C CNN
-F 1 "SW_SPDT" H 2000 8150 50  0000 C CNN
+F 1 "ON/OFF" H 2000 8150 50  0000 C CNN
 F 2 "w_switch:switch_mmp122-r" H 2000 8000 60  0001 C CNN
 F 3 "" H 2000 8000 60  0000 C CNN
@@
 F 0 "C6" H 2500 8010 50  0000 L CNN
 F 1 "C" H 2500 7940 50  0000 L CNN
-F 2 "w_smd_cap:c_0603" H 2450 8000 60  0001 C CNN
+F 2 "w_smd_cap:c_elec_5x5.3" H 2450 8000 60  0001 C CNN
 F 3 "" H 2450 8000 60  0000 C CNN
 	1    2450 8000
 	1    0    0    -1
 $EndComp
-Text Label 2450 7950 0    60   ~ 0
+Text Label 1800 7750 2    60   ~ 0
 12V
 Text Label 2450 8300 0    60   ~ 0
@@
 	2150 7950 2650 7950
 Connection ~ 2450 7950
-Wire Wire Line
-	2250 7750 2250 7950
 Connection ~ 2250 7950
 Wire Wire Line
@@
 P 1550 4550
 F 0 "LD1" H 1550 4650 40  0000 C CNN
-F 1 "LED" H 1600 4450 40  0000 C CNN
+F 1 "LED1" H 1600 4450 40  0000 C CNN
 F 2 "w_smd_leds:Led_0805" H 1550 4550 60  0001 C CNN
 F 3 "" H 1550 4550 60  0000 C CNN
@@
 P 1800 4550
 F 0 "LD2" H 1800 4650 40  0000 C CNN
-F 1 "LED" H 1850 4450 40  0000 C CNN
+F 1 "LED2" H 1850 4450 40  0000 C CNN
 F 2 "w_smd_leds:Led_0805" H 1800 4550 60  0001 C CNN
 F 3 "" H 1800 4550 60  0000 C CNN
@@
 P 2050 4550
 F 0 "LD3" H 2050 4650 40  0000 C CNN
-F 1 "LED" H 2100 4450 40  0000 C CNN
+F 1 "LED3" H 2100 4450 40  0000 C CNN
 F 2 "w_smd_leds:Led_0805" H 2050 4550 60  0001 C CNN
 F 3 "" H 2050 4550 60  0000 C CNN
@@
 P 2300 4550
 F 0 "LD4" H 2300 4650 40  0000 C CNN
-F 1 "LED" H 2350 4450 40  0000 C CNN
+F 1 "LED4" H 2350 4450 40  0000 C CNN
 F 2 "w_smd_leds:Led_0805" H 2300 4550 60  0001 C CNN
 F 3 "" H 2300 4550 60  0000 C CNN
@@
 Text Label 2300 4250 0    60   ~ 0
 LED4
-Text Label 3750 3500 2    60   ~ 0
+Text Label 3750 2600 2    60   ~ 0
 LED1
-Text Label 3750 4100 2    60   ~ 0
+Text Label 3750 2700 2    60   ~ 0
 LED2
-Text Label 3750 4200 2    60   ~ 0
+Text Label 3750 2800 2    60   ~ 0
 LED3
-Text Label 3750 4300 2    60   ~ 0
+Text Label 3750 3300 2    60   ~ 0
 LED4
 Text Label 3750 4400 2    60   ~ 0
@@
 	1    0    0    -1
 $EndComp
-Text Label 2500 1700 2    60   ~ 0
+Text Label 2500 1900 2    60   ~ 0
 SPI1_SCK
 Text Label 2500 1800 2    60   ~ 0
 SPI1_MISO
-Text Label 2500 1900 2    60   ~ 0
+Text Label 2500 1700 2    60   ~ 0
 SPI1_MOSI
 Text Label 2500 2000 2    60   ~ 0
@@
 NoConn ~ 7050 2450
 NoConn ~ 7050 2650
-NoConn ~ 1850 3750
 $Comp
 L R R19
@@
 $EndComp
 $Comp
-L POT R22
+L POT ADC4
 U 1 1 57A0D08D
 P 2400 5350
-F 0 "R22" V 2450 5250 50  0000 C CNN
+F 0 "ADC4" V 2450 5250 50  0000 C CNN
 F 1 "POT" H 2400 5250 50  0001 C CNN
 F 2 "w_pin_strip:pin_socket_3" H 2400 5350 60  0001 C CNN
@@
 Text Label 2400 5500 0    60   ~ 0
 GND
-Text Label 2400 5250 0    60   ~ 0
+Text Label 2450 5250 0    60   ~ 0
 3.3V
 Wire Wire Line
@@
 $EndComp
 $Comp
-L POT R23
+L POT ADC5
 U 1 1 57A0DD3F
 P 2400 5800
-F 0 "R23" V 2450 5700 50  0000 C CNN
+F 0 "ADC5" V 2450 5700 50  0000 C CNN
 F 1 "POT" H 2400 5700 50  0001 C CNN
 F 2 "w_pin_strip:pin_socket_3" H 2400 5800 60  0001 C CNN
@@
 Text Label 2400 5950 0    60   ~ 0
 GND
-Text Label 2400 5700 0    60   ~ 0
+Text Label 2450 5700 0    60   ~ 0
 3.3V
 Wire Wire Line
@@
 $EndComp
 $Comp
-L POT R24
+L POT ADC6
 U 1 1 57A0DF25
 P 2400 6250
-F 0 "R24" V 2450 6150 50  0000 C CNN
+F 0 "ADC6" V 2450 6150 50  0000 C CNN
 F 1 "POT" H 2400 6150 50  0001 C CNN
 F 2 "w_pin_strip:pin_socket_3" H 2400 6250 60  0001 C CNN
@@
 Text Label 2400 6400 0    60   ~ 0
 GND
-Text Label 2400 6150 0    60   ~ 0
+Text Label 2450 6150 0    60   ~ 0
 3.3V
 Wire Wire Line
@@
 Text Label 900  10350 3    60   ~ 0
 GND
+Wire Wire Line
+	2250 7750 1800 7750
+Wire Wire Line
+	1800 7750 1800 8000
+Connection ~ 1800 8000
+Wire Wire Line
+	2400 5250 2450 5250
+Wire Wire Line
+	2400 5700 2450 5700
+Wire Wire Line
+	2400 6150 2450 6150
+$Comp
+L SW_PUSH SW4
+U 1 1 57BD9842
+P 2250 3650
+F 0 "SW4" H 2260 3770 50  0000 C CNN
+F 1 "RESET" H 2250 3570 50  0000 C CNN
+F 2 "w_switch:smd_push" H 2250 3650 60  0001 C CNN
+F 3 "" H 2250 3650 60  0000 C CNN
+	1    2250 3650
+	0    -1   -1   0
+$EndComp
+Text Label 950  4450 0    60   ~ 0
+GND
+Text Label 2200 3500 2    60   ~ 0
+RESET
+Wire Wire Line
+	2200 3500 2250 3500
+Connection ~ 1650 3800
+$Comp
+L HEADER_3 J13
+U 1 1 57BDC9EB
+P 6200 7950
+F 0 "J13" H 6327 8003 60  0000 L CNN
+F 1 "HEADER_3" H 6327 7897 60  0000 L CNN
+F 2 "w_pin_strip:pin_socket_3" H 6200 7950 60  0001 C CNN
+F 3 "" H 6200 7950 60  0000 C CNN
+	1    6200 7950
+	1    0    0    -1
+$EndComp
+$Comp
+L HEADER_3 J14
+U 1 1 57BDCB62
+P 6200 8350
+F 0 "J14" H 6327 8403 60  0000 L CNN
+F 1 "HEADER_3" H 6327 8297 60  0000 L CNN
+F 2 "w_pin_strip:pin_socket_3" H 6200 8350 60  0001 C CNN
+F 3 "" H 6200 8350 60  0000 C CNN
+	1    6200 8350
+	1    0    0    -1
+$EndComp
+$Comp
+L HEADER_3 J15
+U 1 1 57BDCC52
+P 6200 8750
+F 0 "J15" H 6327 8803 60  0000 L CNN
+F 1 "HEADER_3" H 6327 8697 60  0000 L CNN
+F 2 "w_pin_strip:pin_socket_3" H 6200 8750 60  0001 C CNN
+F 3 "" H 6200 8750 60  0000 C CNN
+	1    6200 8750
+	1    0    0    -1
+$EndComp
+Text Label 6100 7850 2    60   ~ 0
+TIM4_CH1
+Text Label 6100 7950 2    60   ~ 0
+TIM4_CH2
+Text Label 6100 8050 2    60   ~ 0
+TIM4_CH3
+Text Label 6100 8250 2    60   ~ 0
+TIM4_CH4
+Text Label 6100 8350 2    60   ~ 0
+TIM2_CH2
+Text Label 6100 8450 2    60   ~ 0
+TIM3_CH2
+Text Label 6100 8650 2    60   ~ 0
+TIM3_CH3
+Text Label 6100 8750 2    60   ~ 0
+TIM3_CH4
+Text Label 6100 8850 2    60   ~ 0
+TIM1_CH1
+NoConn ~ 7050 2550
+$Comp
+L HEADER_3 J16
+U 1 1 57BE2968
+P 6200 9150
+F 0 "J16" H 6327 9203 60  0000 L CNN
+F 1 "I2C2" H 6327 9097 60  0000 L CNN
+F 2 "w_pin_strip:pin_socket_3" H 6200 9150 60  0001 C CNN
+F 3 "" H 6200 9150 60  0000 C CNN
+	1    6200 9150
+	1    0    0    -1
+$EndComp
+Text Label 6100 9050 2    60   ~ 0
+SCL
+Text Label 6100 9150 2    60   ~ 0
+SDA
+Text Label 6100 9250 2    60   ~ 0
+PB12
+Text Label 3750 4100 2    60   ~ 0
+SCL
+Text Label 3750 4200 2    60   ~ 0
+SDA
+Text Label 3750 4300 2    60   ~ 0
+PB12
+NoConn ~ 3750 1200
+NoConn ~ 3750 3500
 $EndSCHEMATC

Commit message: Version 3 PCB
Parts:
- added C10, C11, C8, C9: C, w_smd_cap:c_0603, symbol C
- added D1, D2: SCHOTTKY, w_smd_diode:sod123, symbol SCHOTTKY
- added LD5: RXLED, w_smd_leds:Led_0805, symbol LED
- added LD6: TXLED, w_smd_leds:Led_0805, symbol LED
- added LD7: ON, w_smd_leds:Led_0805, symbol LED
- added R22, R23: R, w_smd_resistors:r_0603, symbol R
- added U2: FT231X, w_smd_qfn:qfn-20, symbol FT231X
- added X1: MINI-USB_SHIELD5P2-32005-601, w_conn_pc:conn_usb_B_mini_smd, symbol MINI-USB_SHIELD5P2-32005-601
- SW1: value SW_PUSH -> SW1
- SW2: value SW_PUSH -> SW2
Connections:
- net labels added: V_USB
- wire segments 60 -> 86
- no-connect marks 9 -> 16
Other:
- moved on the sheet: ADC4, ADC5, ADC6, C1, C2, C3, C4, C5, C6, C7, J1, J10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
